File: Driver Circuit/1R.sch (EAGLE design)
At the start: 20 parts, among them IC1 L298

Commit message: Update 1R.sch
Parts:
- added IC2: ADXL33X, adafruit:ADXL33X
- added JP7: (no value), adafruit:PINHD-1X1
- added U$1, U$3: ARDUINO-BPLACE, adafruit:ARDUINO-BPLACE
- added U$2: X25_168, x25_168:X25_168
Connections:
- new net N$1: C1.1, IC1.VCC, U$1.5V
- new net N$14: IC2.XOUT, U$3.A0
- new net N$15: IC2.YOUT, U$3.A1
- new net N$16: IC2.ZOUT, U$3.A2
- new net N$17: R1.1
- new net N$18: IC2.ST, JP7.1
- new net VS1: IC2.VS, IC2.VS1, U$3.3V
- net GND: now also IC2.GND, IC2.GND1, IC2.GND2, IC2.GND3; no longer R1.1
- net N$10: now also U$2.B-
- net N$11: now also U$2.A+
- net N$12: now also U$2.A-
- net N$13: now also U$2.B+
- net N$3: now also U$1.D13
- net N$4: now also U$1.D12
- net N$5: now also U$1.D11
- net N$7: now also U$1.D9
- net N$8: now also U$1.D8
- net N$9: now also U$1.D10
- net VCC: no longer C1.1, IC1.VCC
