File: Driver Circuit/6R_Complete.sch (EAGLE design)
At the start: 162 parts, among them IC1 L298, IC10 ADXL33X, IC11 ADXL33X, IC12 ADXL33X, IC13 ADXL33X, IC14 ADXL33X, IC15 ADXL33X, IC16 ADXL33X, IC17 ADXL33X, IC18 ADXL33X, IC2 L298, IC3 L298, IC4 L298, IC5 L298, IC6 L298, IC7 ADXL33X, IC8 ADXL33X, IC9 ADXL33X

Commit message: Update 6R_Complete.sch
Parts:
- removed IC10, IC11, IC12, IC7, IC8, IC9: ADXL33X, adafruit:ADXL33X
- removed JP16, JP2, JP23, JP28, JP30, JP35, JP37, JP42, JP43, JP44, JP45, JP46, JP47, JP48, JP8, JP9: (no value), adafruit:PINHD-1X1
Connections:
- removed net N$100: IC11.ZOUT, U$5.A2
- removed net N$101: IC11.ST, JP47.1
- removed net N$102: IC12.YOUT, U$6.A1
- removed net N$103: IC12.XOUT, U$6.A0
- removed net N$104: IC12.ZOUT, U$6.A2
- removed net N$57: D33.A, D37.C, IC5.OUT1, JP31.1
- removed net N$58: D34.A, D38.C, IC5.OUT2, JP32.1, U$11.A+
- removed net N$59: D35.A, D39.C, IC5.OUT3, JP33.1, U$11.A-
- removed net N$73: C1.1, C3.1, C5.1, IC1.VCC, IC2.VCC, IC3.VCC
- removed net N$75: IC12.ST, JP48.1
- removed net N$85: IC7.ST, JP44.1
- removed net N$86: IC8.YOUT, U$2.A1
- removed net N$87: IC8.XOUT, U$2.A0
- removed net N$88: IC8.ZOUT, U$2.A2
- removed net N$89: IC8.ST, JP43.1
- removed net N$90: IC9.YOUT, U$3.A1
- removed net N$91: IC9.XOUT, U$3.A0
- removed net N$92: IC9.ZOUT, U$3.A2
- removed net N$93: IC9.ST, JP45.1
- removed net N$94: IC10.YOUT, U$4.A1
- removed net N$95: IC10.XOUT, U$4.A0
- removed net N$96: IC10.ZOUT, U$4.A2
- removed net N$97: IC10.ST, JP46.1
- removed net N$98: IC11.YOUT, U$5.A1
- removed net N$99: IC11.XOUT, U$5.A0
- net GND: no longer IC10.GND, IC10.GND1, IC10.GND2, IC10.GND3, IC11.GND, IC11.GND1, IC11.GND2, IC11.GND3, IC12.GND, IC12.GND1, IC12.GND2, IC12.GND3, IC7.GND, IC7.GND1, IC7.GND2, IC7.GND3, IC8.GND, IC8.GND1, IC8.GND2, IC8.GND3, IC9.GND, IC9.GND1, IC9.GND2, IC9.GND3, JP28.1, JP35.1, JP42.1, U$11.B-
- net N$60: now also U$11.B-; no longer U$11.B+
- net N$77: no longer JP8.1
- net N$79: now also D33.A, D37.C, IC5.OUT1, JP31.1, U$11.A+; no longer IC7.YOUT, U$1.A1
- net N$83: now also D34.A, D38.C, IC5.OUT2, JP32.1, U$11.A-; no longer IC7.XOUT, U$1.A0
- net N$84: now also D35.A, D39.C, IC5.OUT3, JP33.1, U$11.B+; no longer IC7.ZOUT, U$1.A2
- net VCC: now also C1.1, C3.1, C5.1, IC1.VCC, IC2.VCC, IC3.VCC; no longer JP16.1, JP2.1, JP23.1, JP30.1, JP37.1, JP9.1
- net VS1: no longer IC10.VS, IC10.VS1, IC11.VS, IC11.VS1, IC12.VS, IC12.VS1, IC7.VS, IC7.VS1, IC8.VS, IC8.VS1, IC9.VS, IC9.VS1, U$1.3V, U$2.3V, U$3.3V, U$4.3V, U$5.3V, U$6.3V
